File: RELAY8BASE.brd (EAGLE design)
At the start: 62.2 x 69.8 mm, 76 parts, among them IC1 MCP23017SO, J1 Analog, J2 POWER, J3 Digital_0_7, J4 M100.1, J5 ICSPPTH, J7 PWR SELECT, Q1 2N7002, Q2 2N7002, Q3 2N7002, Q4 2N7002, Q5 2N7002, Q6 2N7002, Q7 2N7002, Q8 2N7002

Commit message: Layout for v1.0 release
Parts:
- removed C1: 100nF, freetronics-original:0603
- removed D1, D2, D3, D4, D5, D6, D7, D8, D9: 1N4004 SMB, freetronics-master-v1.1:SMB-DIODE
- removed IC1: MCP23017SO, microchip:SO28W
- removed JP1, JP2: (no value), freetronics-master-v1:TERMINALBLOCK_3.5MM_8
- removed LED1: CH1/RED, freetronics-master-v1:LED-0603
- removed LED10: PWR/BLUE, freetronics-master-v1:LED-0603
- removed LED2: CH5/RED, freetronics-master-v1:LED-0603
- removed LED3: CH2/RED, freetronics-master-v1:LED-0603
- removed LED4: CH6/RED, freetronics-master-v1:LED-0603
- removed LED5: CH3/RED, freetronics-master-v1:LED-0603
- removed LED6: CH7/RED, freetronics-master-v1:LED-0603
- removed LED7: CH4/RED, freetronics-master-v1:LED-0603
- removed LED8: CH8/RED, freetronics-master-v1:LED-0603
- removed LED9: PWR/GREEN, freetronics-master-v1:LED-0603
- removed Q1, Q2, Q3, Q4, Q5, Q6, Q7, Q8: 2N7002, freetronics-master-v1:SOT23-3
- removed R1, R10, R13, R14, R15, R16, R19, R2, R20, R21, R22, R26, R3, R4, R7, R8, R9: 1K, freetronics-master-v1:0603
- removed R11, R12, R17, R18, R23, R24, R29, R30, R31, R5, R6: 10K, freetronics-master-v1:0603
- removed R25: 2K2, freetronics-master-v1:0603
- removed R27, R28: 4K7, freetronics-master-v1:0603
- removed S1: RESET, freetronics-original:TACTILE_SWITCH_SMD
- removed SJ1, SJ2, SJ3: (no value), freetronics-master-v1.1:SJ_2
- removed SJ4: (no value), freetronics-jon:SJ
- added J10, J14: Analog, freetronics:1X06
- added J11, J15: Digital_0_7, freetronics:1X08
- added J12, J16, J8: M100.1, freetronics-original:1X10
- added J13, J17, J9: POWER, freetronics:1X08
- added J18: External, freetronics:1X06
- added J19, J20: (no value), SparkFun-Connectors:1X04_1MM_RA
- added J21, J22: SMD Grove;4P-2.0-90D;320110032, Connector-new:HW4-SMD-2.0-90D
- J5: value ICSPPTH -> Analog; device freetronics-jon:2X03PTH -> freetronics:1X06
- J6: value (none) -> Digital_0_7; device freetronics-master-v1.1:2X03 -> freetronics:1X08
- J7: value PWR SELECT -> External; device SparkFun:1X02 -> freetronics:1X06
- moved J6 106.7 mm to (118.1, 50.8), flipped to the top, turned to 180 degrees
- moved U$6 74.8 mm to (77.5, 8.64), flipped to the top
- moved J5 53.3 mm to (105.4, 2.54), turned to 0 degrees
- moved J7 35.1 mm to (12.7, 33.0)
- moved JP3 12.5 mm to (67.3, 16.5), turned to 0 degrees
Connections:
- removed net 12V: D1.C, D2.C, D3.C, D4.C, D5.C, D6.C, D7.C, D8.C, D9.C, J7.1, JP1.2, JP1.4, JP1.6, JP1.8, JP2.2, JP2.4, JP2.6, JP2.8, LED1.A, LED2.A, LED3.A, LED4.A, LED5.A, LED6.A, LED7.A, LED8.A, R25.2
- removed net 3V3: J2.4
- removed net 5V: J2.5, SJ4.2
- removed net A0: J1.1
- removed net A1: J1.2
- removed net A2: J1.3
- removed net A3: J1.4
- removed net A4_SDA: J1.5, SJ2.1
- removed net A5_SCL: J1.6, SJ1.1
- removed net ADDR0: IC1.15, J6.2, R29.2
- removed net ADDR1: IC1.16, J6.4, R30.2
- removed net ADDR2: IC1.17, J6.6, R31.2
- removed net AREF: J4.8
- removed net D0_RX: J3.1
- removed net D10: J4.3
- removed net D11_MOSI: J4.4
- removed net D12_MISO: J4.5
- removed net D13_SCK: J4.6
- removed net D1_TX: J3.2
- removed net D2: J3.3
- removed net D3: J3.4
- removed net D4: J3.5
- removed net D5: J3.6
- removed net D6: J3.7
- removed net D7: J3.8
- removed net D8: J4.1
- removed net D9: J4.2
- removed net GPA0: IC1.21, R3.2
- removed net GPA1: IC1.22, R9.2
- removed net GPA2: IC1.23, R15.2
- removed net GPA3: IC1.24, R21.2
- removed net GPA4: IC1.25, R4.2
- removed net GPA5: IC1.26, R10.2
- removed net GPA6: IC1.27, R16.2
- removed net GPA7: IC1.28, R22.2
- removed net N$1: Q1.1, R3.1, R5.2
- removed net N$10: Q5.1, R15.1, R17.2
- removed net N$11: D7.A, JP1.1, Q7.3, R19.2
- removed net N$12: Q7.1, R21.1, R23.2
- removed net N$13: D2.A, JP2.7, Q2.3, R2.2
- removed net N$14: Q2.1, R4.1, R6.2
- removed net N$15: D4.A, JP2.5, Q4.3, R8.2
- removed net N$16: Q4.1, R10.1, R12.2
- removed net N$17: D6.A, JP2.3, Q6.3, R14.2
- removed net N$18: Q6.1, R16.1, R18.2
- removed net N$19: D8.A, JP2.1, Q8.3, R20.2
- removed net N$20: Q8.1, R22.1, R24.2
- removed net N$21: LED3.C, R7.1
- removed net N$22: LED7.C, R19.1
- removed net N$23: LED5.C, R13.1
- removed net N$24: LED1.C, R1.1
- removed net N$25: LED2.C, R2.1
- removed net N$26: LED4.C, R8.1
- removed net N$27: LED6.C, R14.1
- removed net N$28: LED8.C, R20.1
- removed net N$3: D3.A, JP1.5, Q3.3, R7.2
- removed net N$4: LED9.A, R25.1
- removed net N$41: D9.A, JP3.1
- removed net N$42: R27.2, SJ3.3
- removed net N$43: R28.2, SJ3.1
- removed net N$5: D1.A, JP1.7, Q1.3, R1.2
- removed net N$52: LED10.A, R26.1
- removed net N$8: Q3.1, R11.2, R9.1
- removed net N$9: D5.A, JP1.3, Q5.3, R13.2
- removed net NC: J2.1
- removed net R3_SCL: J4.10, SJ1.3
- removed net R3_SDA: J4.9, SJ2.3
- removed net RESET: IC1.18, J2.3, S1.3, S1.4
- new net !RESET: J13.3, J17.3, J18.1, J2.3, J7.1, J9.3
- net GND: now also J12.7, J13.6, J13.7, J16.7, J17.6, J17.7, J18.6, J19.1, J20.1, J21.4, J21.SS1, J21.SS2, J22.4, J22.SS1, J22.SS2, J7.6, J8.7, J9.6, J9.7; no longer C1.2, IC1.10, LED10.C, LED9.C, Q1.2, Q2.2, Q3.2, Q4.2, Q5.2, Q6.2, Q7.2, Q8.2, R11.1, R12.1, R17.1, R18.1, R23.1, R24.1, R29.1, R30.1, R31.1, R5.1, R6.1, S1.1, S1.2
- net IOREF: now also J13.2, J17.2, J18.4, J19.2, J20.2, J21.3, J22.3, J7.4, J9.2; no longer C1.1, IC1.9, J6.1, J6.3, J6.5, R26.2, SJ3.2, SJ4.1
- net SCL: now also J12.10, J16.10, J18.3, J19.4, J20.4, J21.1, J22.1, J4.10, J7.3, J8.10; no longer IC1.12, R27.1, SJ1.2
- net SDA: now also J12.9, J16.9, J18.2, J19.3, J20.3, J21.2, J22.2, J4.9, J7.2, J8.9; no longer IC1.13, R28.1, SJ2.2
- net VIN: now also J13.8, J17.8, J18.5, J7.5, J9.8, JP3.1; no longer J7.2
Routing:
- net SCL: track 13.8 -> 514.7 mm, vias 1 -> 5
- net SDA: track 13.2 -> 460.3 mm, vias 1 -> 4
- net IOREF: track 49.0 -> 407.7 mm, vias 1 -> 4
- net !RESET: track 0.00 -> 344.0 mm, vias 0 -> 4
- net VIN: track 5.08 -> 310.5 mm
- net 12V: track 248.3 -> 0.00 mm, vias 8 -> 0
- net GPA7: track 65.3 -> 0.00 mm
- net A4_SDA: track 62.3 -> 0.00 mm
- net GPA6: track 60.1 -> 0.00 mm
- net GPA5: track 54.9 -> 0.00 mm
- net A5_SCL: track 54.8 -> 0.00 mm
- net GPA4: track 49.7 -> 0.00 mm
- net GPA3: track 44.5 -> 0.00 mm
- net GPA2: track 39.3 -> 0.00 mm
- net N$3: track 35.6 -> 0.00 mm, vias 2 -> 0
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Other:
- board size 62.2 x 69.8 mm -> 245.1 x 53.3 mm
- board text added: "!RESET"
- board text added: "(c) 2019 SuperHouse Automation"
- board text added: "+"
- board text added: "-"
- board text added: "Grove"
- board text added: "Qwiic"
- board text added: "Relay Shield Carrier"
- board text added: "SKU: RSC"
- board text added: "v1.0"
- board text added: "www.superhouse.tv/rsc"
- board text removed: "&"
- board text removed: "(c) 2012-14 Freetronics Pty Ltd"
- board text removed: "0 0 0 0 1 1 1 1"
- board text removed: "0 0 1 1 0 0 1 1"
- board text removed: "0 1 0 1 0 1 0 1"
- board text removed: "0x20 0x21 0x22 0x23 0x24 0x25 0x26 0x27"
- board text removed: "1"
- board text removed: "2"
- board text removed: "3"
- board text removed: "3.3V"
- board text removed: "3V3"
- board text removed: "4"
- board text removed: "5"
- board text removed: "5-24Vdc IN"
- board text removed: "5V"
- board text removed: "6"
- board text removed: "7"
- board text removed: "8"
- board text removed: "8-Channel Relay Driver Shield"
- board text removed: "8-Channel Relay Driver Shield v2.0"
- board text removed: "A"
- board text removed: "A0"
- board text removed: "A1"
- board text removed: "A2"
- board text removed: "A3"
- board text removed: "A4"
- board text removed: "A5"
- board text removed: "COMPATIBLE"
- board text removed: "D0"
- board text removed: "D1"
- board text removed: "D10"
- board text removed: "D11"
- board text removed: "D12"
- board text removed: "D13"
- board text removed: "D2"
- board text removed: "D3"
- board text removed: "D4"
- board text removed: "D5"
- board text removed: "D6"
- board text removed: "D7"
- board text removed: "D8"
- board text removed: "D9"
- board text removed: "DC"
- board text removed: "HEX"
- board text removed: "I2C ADDR"
- board text removed: "I2C ADDRESS"
- board text removed: "I2C PIN SELECT"
- board text removed: "INPUT"
- board text removed: "K"
- board text removed: "LINK"
- board text removed: "MCP23017"
- board text removed: "OUT"
- board text removed: "PULLUPS"
- board text removed: "PWR"
- board text removed: "R1/2"
- board text removed: "R3"
- board text removed: "RESET"
- board text removed: "ROHS"
- board text removed: "SKU: RELAY8"
- board text removed: "TO 5V"
- board text removed: "freetronics"
- board text removed: "tron.cc/r8"
- board text removed: "www.freetronics.com"
- board text removed: "www.freetronics.com/relay8"
