File: RSC.brd (EAGLE design)
At the start: 245.1 x 53.3 mm, 24 parts, among them J1 Analog, J10 Analog, J11 Digital_0_7, J12 M100.1, J13 POWER, J14 Analog, J15 Digital_0_7, J16 M100.1, J17 POWER, J18 External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

Commit message: Changed designators to make them sequential
Parts:
- renumbered J1 to H2, J10 to H10, J11 to H12, J12 to H11, J13 to H9, J14 to H14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
